File: _autosave-weather.kicad_sch (KiCad schematic)
At the start: 31 parts, among them J1 Conn_01x09_Socket, J2 BreakoutOfTemp+humid+pressure, Q3 AO3400A, Q4 AO3400A, U1 DRA818V, U3 DS18B20, U5 INA180A3, U7 4554, U8 TPS563200

Commit message: polishing schematic and laying out PCB
Parts:
- R7: footprint (none) -> Connector_PinSocket_2.54mm:PinSocket_1x02_P2.54mm_Vertical
- U3: footprint Package_TO_SOT_THT:TO-92_Inline -> Connector_PinSocket_2.54mm:PinSocket_1x03_P2.54mm_Vertical
Connections:
- net +3.3V: now also U4.9 (3.3v)
- no-connect marks 13 -> 18
