File: weather.kicad_pcb (KiCad board)
At the start: 2 copper layers, 94.5 x 68 mm, 14 parts, among them J1 Conn_01x09_Socket, Q1 2N7002H, Q2 2N7002H, U1 DRA818V, U2 TPS62132, U3 DS18B20, U4 DS18B20, U5 BMP280

Commit message: PCB layout preview
Parts:
- removed BT1: 7.4, Connector_PinSocket_2.54mm:PinSocket_1x02_P2.54mm_Vertical
- removed Q1, Q2: 2N7002H, Package_TO_SOT_SMD:SOT-23
- removed U2: TPS62132, Package_DFN_QFN:VQFN-16-1EP_3x3mm_P0.5mm_EP1.68x1.68mm_ThermalVias
- added C5: 3300uf, Capacitor_THT:CP_Radial_D12.5mm_P5.00mm, F.Cu at (126.0, 123.9)
- added C8: 100nf, Capacitor_SMD:C_0805_2012Metric_Pad1.18x1.45mm_HandSolder, F.Cu at (108.7, 93.1)
- added CfirstBat1: 10uF, Capacitor_SMD:C_0805_2012Metric_Pad1.18x1.45mm_HandSolder, F.Cu at (101.0, 88.5)
- added CforSD1: 100nf, Capacitor_SMD:C_0805_2012Metric_Pad1.18x1.45mm_HandSolder, F.Cu at (132.2, 107.8)
- added CoutputCap1: 22uf, Capacitor_SMD:C_0805_2012Metric_Pad1.18x1.45mm_HandSolder, F.Cu at (115.8, 93.1)
- added J2: BreakoutOfTemp+humid+pressure, Connector_PinSocket_2.54mm:PinSocket_1x07_P2.54mm_Vertical, F.Cu at (61.9, 87.4)
- added L2: 2.2uH, Inductor_SMD:L_0805_2012Metric_Pad1.05x1.20mm_HandSolder, F.Cu at (111.1, 93.1)
- added Q3: AO3400A, Package_TO_SOT_SMD:SOT-23, F.Cu at (121.7, 113.4)
- added Q4: AO3400A, Package_TO_SOT_SMD:SOT-23, F.Cu at (134.5, 129.9)
- added R10: 10k, Resistor_SMD:R_0805_2012Metric_Pad1.20x1.40mm_HandSolder, F.Cu at (113.5, 88.8)
- added R4: 5k, Resistor_SMD:R_0805_2012Metric_Pad1.20x1.40mm_HandSolder, F.Cu at (58.1, 138.6)
- added R5: 10k, Resistor_SMD:R_0805_2012Metric_Pad1.20x1.40mm_HandSolder, F.Cu at (58.1, 141.6)
- added R6: 10k, Resistor_SMD:R_0805_2012Metric_Pad1.20x1.40mm_HandSolder, F.Cu at (87.9, 125.7)
- added R8: 1klook at again tho, Resistor_SMD:R_0805_2012Metric_Pad1.20x1.40mm_HandSolder, F.Cu at (122.2, 136.7)
- added R9: 34k, Resistor_SMD:R_0805_2012Metric_Pad1.20x1.40mm_HandSolder, F.Cu at (113.4, 93.1)
- added U7: 4554, 4554:MODULE_4554, F.Cu at (82.7, 94.3)
- added U8: TPS563200, Package_TO_SOT_SMD:SOT-23-6, F.Cu at (105.0, 92.9)
- R2: value 5k -> .01
- R3: value R -> 39
- SC1: footprint Connector_PinSocket_2.54mm:PinSocket_1x02_P2.54mm_Vertical -> TestPoint:TestPoint_2Pads_Pitch5.08mm_Drill1.3mm
- U1: footprint LightAPRS:PinSocket_1x10_P2.54mm_Vertical -> VHF_UHF_Modules:VHF_UHF_Module_generic
- U4: value DS18B20 -> ~; footprint Package_TO_SOT_THT:TO-92_Inline -> PCM_SparkFun-GNSS:SparkFun GNSS Receiver Breakout - MAX-M10S (Qwiic)
- U5: value BMP280 -> INA180A3; footprint Package_LGA:Bosch_LGA-8_2x2.5mm_P0.65mm_ClockwisePinNumbering -> Package_TO_SOT_SMD:SOT-23-5
- moved U4 97.1 mm to (54.3, 57.6)
- moved R1 49.4 mm to (58.1, 132.7), turned to 0 degrees
- moved U5 38.9 mm to (121.7, 106.5)
- moved U1 37.2 mm to (77.1, 154.6), turned to 90 degrees
- moved U3 29.7 mm to (81.7, 113.4)
- moved R2 28.3 mm to (121.6, 109.8)
- moved J1 25.2 mm to (161.7, 143.2), turned to 0 degrees
- moved SC1 13.4 mm to (128.3, 132.1)
- moved A1 12.9 mm to (107.5, 128.4)
- moved R3 6.23 mm to (139.1, 129.2), turned to 180 degrees
Connections:
- A1 pad 1: Net-(A1-GPIO0) -> /SDA0
- A1 pad 10: unconnected-(A1-GPIO7-Pad10) -> Net-(A1-GPIO7)
- A1 pad 17: Net-(A1-GPIO13) -> unconnected-(A1-GPIO13-Pad17)
- A1 pad 19: Net-(A1-GPIO14) -> unconnected-(A1-GPIO14-Pad19)
- A1 pad 2: Net-(A1-GPIO1) -> /SCL0
- A1 pad 31: unconnected-(A1-GPIO26_ADC0-Pad31) -> /ADC0
- A1 pad 32: Net-(A1-GPIO27_ADC1) -> /ADC1
- A1 pad 34: Net-(A1-GPIO28_ADC2) -> /ADC2
- A1 pad 36: unconnected-(A1-3V3-Pad36)_1 -> /pico3.3
- A1 pad 4: Net-(A1-GPIO2) -> /SDA
- A1 pad 5: Net-(A1-GPIO3) -> /SCL1
- A1 pad 6: unconnected-(A1-GPIO4-Pad6) -> /Pin6GP4
- A1 pad 7: unconnected-(A1-GPIO5-Pad7) -> Net-(A1-GPIO5)
- A1 pad 9: unconnected-(A1-GPIO6-Pad9) -> Net-(A1-GPIO6)
- J1 pad 1: +3.3V pico -> +3.3V
- R1 pad 1: +3.3V pico -> +3.3V
- R1 pad 2: Net-(A1-GPIO13) -> Net-(A1-GPIO5)
- R2 pad 1: Net-(A1-GPIO14) -> GND
- R2 pad 2: +3.3V -> Net-(Q3-S)
- SC1 pad 1: Net-(A1-GPIO28_ADC2) -> /ADC1
- U1 pad 1: Net-(A1-GPIO2) -> Net-(A1-GPIO7)
- U1 pad 6: Net-(A1-GPIO13) -> Net-(A1-GPIO5)
- U1 pad 7: Net-(A1-GPIO3) -> Net-(A1-GPIO6)
- U4 pad 1: GND -> (no net)
- U4 pad 2: Net-(A1-GPIO14) -> (no net)
- U4 pad 3: +3.3V -> (no net)
- U5 pad 1: GND -> /ADC2
- U5 pad 2: +3.3V -> GND
- U5 pad 3: Net-(A1-GPIO0) -> Net-(Q3-S)
- U5 pad 4: Net-(A1-GPIO1) -> GND
- U5 pad 5: GND -> +3.3V
Routing:
- net (no net): track 61.4 -> 0.00 mm
- net Net-(A1-VSYS): track 54.3 -> 0.00 mm
- net /ADC1: track 0.00 -> 36.2 mm
- net Net-(A1-GPIO17): track 0.00 -> 33.5 mm, vias 0 -> 1
- net Net-(A1-GPIO21): track 0.00 -> 30.2 mm, vias 0 -> 1
- net Net-(A1-GPIO20): track 29.8 -> 0.00 mm
- net unconnected-(A1-GPIO7-Pad10): track 26.7 -> 0.00 mm
- net Net-(A1-GPIO8): track 26.7 -> 0.00 mm
- net Net-(BT1-+): track 25.6 -> 0.00 mm
- net /ADC2: track 0.00 -> 17.5 mm, vias 0 -> 1
- net Net-(A1-GPIO16): track 15.9 -> 0.00 mm
- net Net-(U2-ADJ): track 15.3 -> 0.00 mm
- net /VFB: track 0.00 -> 13.0 mm
- net Net-(A1-GPIO19): track 11.0 -> 0.00 mm
- net Net-(A1-GPIO18): track 11.0 -> 0.00 mm
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- added copper zone on In2.Cu, net +3.3V
- added copper zone on In1.Cu, net GND
- removed copper zone on B.Cu, net GND
Other:
- board outline removed
- copper layers 2 -> 4

Commit message: minor bug fixes
Parts:
- added AE1: Antenna, Connector_Coaxial:SMA_Amphenol_132289_EdgeMount, F.Cu at (45.7, 149.2)
- added R7: R_Photo, Connector_PinSocket_2.54mm:PinSocket_1x02_P2.54mm_Vertical, F.Cu at (163.2, 127.8)
- U3: footprint Package_TO_SOT_THT:TO-92_Inline -> Connector_PinSocket_2.54mm:PinSocket_1x03_P2.54mm_Vertical
- moved U7 93.4 mm to (137.4, 170.1), turned to 180 degrees
- moved CforSD1 38.8 mm to (158.2, 136.6), turned to 180 degrees
- moved R8 37.0 mm to (158.0, 127.6)
- moved U4 28.1 mm to (80.6, 67.4)
- moved R1 27.7 mm to (83.5, 143.7)
- moved R4 27.7 mm to (83.5, 149.6)
- moved R5 27.7 mm to (83.5, 152.6)
- moved U1 18.6 mm to (63.6, 141.9), turned to -90 degrees
- moved CoutputCap1 17.7 mm to (132.4, 99.5)
- moved L2 17.7 mm to (127.7, 99.5)
- moved C8 17.7 mm to (125.2, 99.5)
- moved CfirstBat1 17.7 mm to (117.5, 94.8)
- moved R10 17.7 mm to (130.1, 95.1)
- moved U8 17.7 mm to (121.5, 99.3)
- moved R9 17.7 mm to (129.9, 99.5)
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Connections:
- CforSD1 pad 1: unconnected-(CforSD1-Pad1) -> GND
- CforSD1 pad 2: unconnected-(CforSD1-Pad2) -> +3.3V
- U4 pad 9: unconnected-(U4-3.3v-Pad9) -> +3.3V
Routing:
- net Net-(Q3-D): track 6.40 -> 0.25 mm
- net GND: track 8.51 -> 13.1 mm, vias 3 -> 7
- net /bat: track 6.19 -> 8.86 mm
- net Net-(A1-GPIO17): track 33.5 -> 36.1 mm
- net /ADC2: track 17.5 -> 18.5 mm
- net /ADC1: track 36.2 -> 37.1 mm
- net Net-(A1-GPIO21): track 30.2 -> 31.1 mm

Commit message: PCB layout
Parts:
- moved R7 72.1 mm to (91.2, 123.5), turned to 0 degrees
- moved R8 67.0 mm to (91.1, 131.1), turned to -90 degrees
- moved U3 59.6 mm to (105.2, 167.0), turned to 180 degrees
- moved U4 20.0 mm to (65.1, 80.0), turned to 180 degrees
- moved R4 19.4 mm to (99.4, 160.6), turned to 180 degrees
- moved R1 18.3 mm to (79.0, 161.4), turned to 180 degrees
- moved R6 16.3 mm to (77.8, 138.5), turned to 180 degrees
- moved AE1 16.1 mm to (44.7, 165.2)
- moved J2 15.1 mm to (63.4, 107.7)
- moved U7 10.7 mm to (136.9, 180.8)
- moved U1 10.0 mm to (63.5, 151.9)
- moved R9 8.01 mm to (131.0, 91.5)
- moved C8 8.01 mm to (126.2, 91.5)
- moved CfirstBat1 8.01 mm to (118.5, 86.9)
- moved U8 8.01 mm to (122.6, 91.3)
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Connections:
- R7 pad 1: /pico3.3 -> +3.3V
Routing:
- net /SDA: track 0.00 -> 114.7 mm, vias 0 -> 1
- net /SCL1: track 0.00 -> 110.9 mm
- net Net-(A1-GPIO22): track 0.41 -> 75.2 mm
- net Net-(A1-GPIO6): track 0.00 -> 57.7 mm, vias 0 -> 2
- net Net-(A1-GPIO5): track 0.00 -> 57.3 mm, vias 0 -> 1
- net /Pin6GP4: track 0.00 -> 52.4 mm
- net Net-(A1-GPIO8): track 0.00 -> 52.1 mm, vias 0 -> 2
- net Net-(A1-GPIO19): track 0.00 -> 48.9 mm, vias 0 -> 2
- net Net-(A1-GPIO9): track 0.00 -> 47.6 mm
- net Net-(A1-GPIO18): track 0.00 -> 46.0 mm, vias 0 -> 2
- net Net-(A1-GPIO20): track 0.00 -> 44.2 mm
- net Net-(A1-GPIO16): track 0.00 -> 41.0 mm
- net /SDA0: track 0.00 -> 38.6 mm
- net GND: track 13.1 -> 48.7 mm, vias 7 -> 26
- net /SCL0: track 0.00 -> 34.8 mm
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